File: src/kicad/2 EQ Piezo preamp.sch (KiCad schematic (older format))
At the start: 26 parts, among them P1 IN, P2 OUT, P3 9V, U1 OPA2244

Commit message: latest mods
Signed-off-by: Badscrew <badscrew@dolganoff.com>
Parts:
- C1, C11, C4, C5, C6, C7: symbol C -> C-RESCUE-2_EQ_Piezo_preamp
- C10, C3, C8, C9: symbol CP1 -> CP1-RESCUE-2_EQ_Piezo_preamp
- R1, R2, R3, R4, R5, R6, R7, R8, R9: symbol R -> R-RESCUE-2_EQ_Piezo_preamp
Changed lines of the file:
@@
 EESchema Schematic File Version 2
+LIBS:2 EQ Piezo preamp-rescue
 LIBS:power
 LIBS:device
@@
 LIBS:memory
 LIBS:xilinx
-LIBS:special
 LIBS:microcontrollers
 LIBS:dsp
@@
 $EndComp
 $Comp
-L R R4
+L R-RESCUE-2_EQ_Piezo_preamp R4
 U 1 1 535928BD
 P 5000 2950
@@
 $EndComp
 $Comp
-L R R5
+L R-RESCUE-2_EQ_Piezo_preamp R5
 U 1 1 535928EA
 P 5000 3550
@@
 $EndComp
 $Comp
-L R R6
+L R-RESCUE-2_EQ_Piezo_preamp R6
 U 1 1 53592917
 P 5600 2450
@@
 $EndComp
 $Comp
-L R R3
+L R-RESCUE-2_EQ_Piezo_preamp R3
 U 1 1 53592926
 P 4700 2900
@@
 	5000 2600 5000 2700
 $Comp
-L C C5
+L C-RESCUE-2_EQ_Piezo_preamp C5
 U 1 1 535929E0
 P 5000 2100
@@
 	5000 3900 5000 3800
 $Comp
-L C C6
+L C-RESCUE-2_EQ_Piezo_preamp C6
 U 1 1 53592A4C
 P 5600 4050
@@
 $EndComp
 $Comp
-L C C4
+L C-RESCUE-2_EQ_Piezo_preamp C4
 U 1 1 53592A5B
 P 4700 3550
@@
 Connection ~ 6950 3150
 $Comp
-L C C7
+L C-RESCUE-2_EQ_Piezo_preamp C7
 U 1 1 53592AE6
 P 6450 3800
@@
 Connection ~ 6950 3800
 $Comp
-L R R7
+L R-RESCUE-2_EQ_Piezo_preamp R7
 U 1 1 53592B29
 P 7200 3500
@@
 $EndComp
 $Comp
-L CP1 C9
+L CP1-RESCUE-2_EQ_Piezo_preamp C9
 U 1 1 53592B91
 P 7650 3500
@@
 Vref
 $Comp
-L GND #PWR01
+L GND-RESCUE-2_EQ_Piezo_preamp #PWR01
 U 1 1 53592BEB
 P 6300 3550
@@
 	7850 3500 7950 3500
 $Comp
-L GND #PWR03
+L GND-RESCUE-2_EQ_Piezo_preamp #PWR03
 U 1 1 53592D0A
 P 8050 4250
@@
 $EndComp
 $Comp
-L GND #PWR05
+L GND-RESCUE-2_EQ_Piezo_preamp #PWR05
 U 1 1 53592DB8
 P 3400 3650
@@
 $EndComp
 $Comp
-L R R2
+L R-RESCUE-2_EQ_Piezo_preamp R2
 U 1 1 53592DBE
 P 2950 2850
@@
 Vref
 $Comp
-L C C1
+L C-RESCUE-2_EQ_Piezo_preamp C1
 U 1 1 53592E16
 P 2700 3150
@@
 $EndComp
 $Comp
-L R R1
+L R-RESCUE-2_EQ_Piezo_preamp R1
 U 1 1 53592E1C
 P 2200 3150
@@
 	1950 3350 1950 3450
 $Comp
-L GND #PWR06
+L GND-RESCUE-2_EQ_Piezo_preamp #PWR06
 U 1 1 53592F22
 P 1950 3450
@@
 $EndComp
 $Comp
-L R R8
+L R-RESCUE-2_EQ_Piezo_preamp R8
 U 1 1 53592F97
 P 7600 1950
@@
 $EndComp
 $Comp
-L R R9
+L R-RESCUE-2_EQ_Piezo_preamp R9
 U 1 1 53592F9D
 P 7600 2550
@@
 $EndComp
 $Comp
-L CP1 C8
+L CP1-RESCUE-2_EQ_Piezo_preamp C8
 U 1 1 53592FA3
 P 7300 2550
@@
 $EndComp
 $Comp
-L CP1 C10
+L CP1-RESCUE-2_EQ_Piezo_preamp C10
 U 1 1 53592FA9
 P 7800 2250
@@
 	7800 1650 7800 2050
 $Comp
-L C C11
+L C-RESCUE-2_EQ_Piezo_preamp C11
 U 1 1 53593118
 P 8050 2650
@@
 Connection ~ 6950 3500
 $Comp
-L GND #PWR07
+L GND-RESCUE-2_EQ_Piezo_preamp #PWR07
 U 1 1 53593251
 P 7600 2900
@@
 	4700 4050 4750 4050
 $Comp
-L CP1 C3
+L CP1-RESCUE-2_EQ_Piezo_preamp C3
 U 1 1 53593897
 P 4250 3250
